Commit message: Update XFL201 supplier vehicle parameters

File: forklift_nav2_demo/urdf/xfl201_steered.urdf.xacro (robot description, xacro)
@@ -3,7 +3,7 @@
   <xacro:arg name="gazebo_cmd_vel_topic" default="cmd_vel"/>
   <xacro:arg name="gazebo_scan_topic" default="scan"/>
-  <xacro:property name="wheel_radius" value="0.15"/>
+  <xacro:property name="wheel_radius" value="0.225"/>
   <xacro:property name="wheel_width" value="0.08"/>
-  <xacro:property name="wheel_separation" value="0.86"/>
+  <xacro:property name="wheel_separation" value="0.936"/>
   <xacro:property name="base_z" value="0.22"/>
   <xacro:property name="body_length" value="2.10"/>
@@ -124,5 +124,5 @@
     <parent link="base_link"/>
     <child link="left_wheel_link"/>
-    <origin xyz="0 ${wheel_separation / 2.0} -0.06" rpy="0 0 0"/>
+    <origin xyz="0 ${wheel_separation / 2.0} ${wheel_radius - base_z}" rpy="0 0 0"/>
     <axis xyz="0 1 0"/>
   </joint>
@@ -150,5 +150,5 @@
     <parent link="base_link"/>
     <child link="right_wheel_link"/>
-    <origin xyz="0 ${-wheel_separation / 2.0} -0.06" rpy="0 0 0"/>
+    <origin xyz="0 ${-wheel_separation / 2.0} ${wheel_radius - base_z}" rpy="0 0 0"/>
     <axis xyz="0 1 0"/>
   </joint>
