Commit message: feat: harden real-vehicle navigation and pallet approach
Add external-localization, fine-motion, and pallet-approach adapters.

Improve A* path shaping, pivot execution, MPC transitions, safety gating, and Curtis odometry handling.

Add real-vehicle configs, RViz views, diagnostics, deployment guides, and focused tests.

File: forklift_nav2_demo/urdf/forklift_diff_drive.urdf.xacro (robot description, xacro)
@@ -195,5 +195,5 @@
     <parent link="base_link"/>
     <child link="base_scan"/>
-    <origin xyz="0.25 0 0.30" rpy="0 0 0"/>
+    <origin xyz="0 0 0" rpy="0 0 0"/>
   </joint>
   <gazebo reference="base_link">

Commit message: fix(navigation): stabilize segmented planning and MPC tracking

File: forklift_nav2_demo/urdf/forklift_diff_drive.urdf.xacro (robot description, xacro)
@@ -3,8 +3,19 @@
   <xacro:arg name="gazebo_cmd_vel_topic" default="cmd_vel"/>
   <xacro:arg name="gazebo_scan_topic" default="scan"/>
-  <xacro:property name="wheel_radius" value="0.16"/>
-  <xacro:property name="wheel_width" value="0.08"/>
-  <xacro:property name="wheel_separation" value="0.76"/>
-  <xacro:property name="base_z" value="0.22"/>
+  <!-- 2MKC20M30LV205 geometry. base_link is the drive-axle center and -X points to the forks. -->
+  <xacro:property name="drive_wheel_radius" value="0.2285"/>
+  <xacro:property name="drive_wheel_width" value="0.178"/>
+  <xacro:property name="drive_track_width" value="0.937"/>
+  <xacro:property name="support_wheel_radius" value="0.1905"/>
+  <xacro:property name="support_wheel_width" value="0.127"/>
+  <xacro:property name="support_track_width" value="0.183"/>
+  <xacro:property name="wheel_base" value="1.40"/>
+  <xacro:property name="base_z" value="${drive_wheel_radius}"/>
+  <xacro:property name="body_length" value="2.079"/>
+  <xacro:property name="body_width" value="1.220"/>
+  <xacro:property name="body_center_x" value="0.6695"/>
+  <xacro:property name="mast_x" value="-0.370"/>
+  <xacro:property name="fork_length" value="1.220"/>
+  <xacro:property name="fork_center_x" value="-0.980"/>
   <link name="base_footprint"/>
   <joint name="base_joint" type="fixed">
@@ -15,12 +26,12 @@
   <link name="base_link">
     <inertial>
-      <origin xyz="0 0 0"/>
+      <origin xyz="${body_center_x} 0 0"/>
       <mass value="28.0"/>
       <inertia ixx="1.20" ixy="0.0" ixz="0.0" iyy="3.40" iyz="0.0" izz="3.80"/>
     </inertial>
     <visual name="body_visual">
-      <origin xyz="0 0 0" rpy="0 0 0"/>
-      <geometry>
-        <box size="1.685 1.16 0.28"/>
+      <origin xyz="${body_center_x} 0 0" rpy="0 0 0"/>
+      <geometry>
+        <box size="${body_length} ${body_width} 0.26"/>
       </geometry>
       <material name="forklift_yellow">
@@ -29,13 +40,13 @@
     </visual>
     <collision name="body_collision">
-      <origin xyz="0 0 0" rpy="0 0 0"/>
-      <geometry>
-        <box size="1.685 1.16 0.28"/>
+      <origin xyz="${body_center_x} 0 0" rpy="0 0 0"/>
+      <geometry>
+        <box size="${body_length} ${body_width} 0.26"/>
       </geometry>
     </collision>
     <visual name="counterweight_visual">
-      <origin xyz="0.73 0 0.02" rpy="0 0 0"/>
-      <geometry>
-        <box size="0.24 1.06 0.34"/>
+      <origin xyz="1.55 0 0.02" rpy="0 0 0"/>
+      <geometry>
+        <box size="0.318 1.12 0.34"/>
       </geometry>
       <material name="dark_gray">
@@ -44,13 +55,13 @@
     </visual>
     <collision name="counterweight_collision">
-      <origin xyz="0.73 0 0.02" rpy="0 0 0"/>
-      <geometry>
-        <box size="0.24 1.06 0.34"/>
+      <origin xyz="1.55 0 0.02" rpy="0 0 0"/>
+      <geometry>
+        <box size="0.318 1.12 0.34"/>
       </geometry>
     </collision>
     <visual name="mast_visual">
-      <origin xyz="-0.843 0 0.30" rpy="0 0 0"/>
-      <geometry>
-        <box size="0.10 0.95 0.82"/>
+      <origin xyz="${mast_x} 0 0.835" rpy="0 0 0"/>
+      <geometry>
+        <box size="0.10 0.97 1.917"/>
       </geometry>
       <material name="mast_gray">
@@ -59,13 +70,13 @@
     </visual>
     <collision name="mast_collision">
-      <origin xyz="-0.843 0 0.30" rpy="0 0 0"/>
-      <geometry>
-        <box size="0.10 0.95 0.82"/>
+      <origin xyz="${mast_x} 0 0.835" rpy="0 0 0"/>
+      <geometry>
+        <box size="0.10 0.97 1.917"/>
       </geometry>
     </collision>
     <visual name="fork_left_visual">
-      <origin xyz="-1.443 0.25 -0.13" rpy="0 0 0"/>
-      <geometry>
-        <box size="1.20 0.10 0.04"/>
+      <origin xyz="${fork_center_x} 0.25 -0.1885" rpy="0 0 0"/>
+      <geometry>
+        <box size="${fork_length} 0.10 0.04"/>
       </geometry>
       <material name="fork_gray">
@@ -74,20 +85,20 @@
     </visual>
     <collision name="fork_left_collision">
-      <origin xyz="-1.443 0.25 -0.13" rpy="0 0 0"/>
-      <geometry>
-        <box size="1.20 0.10 0.04"/>
+      <origin xyz="${fork_center_x} 0.25 -0.1885" rpy="0 0 0"/>
+      <geometry>
+        <box size="${fork_length} 0.10 0.04"/>
       </geometry>
     </collision>
     <visual name="fork_right_visual">
-      <origin xyz="-1.443 -0.25 -0.13" rpy="0 0 0"/>
-      <geometry>
-        <box size="1.20 0.10 0.04"/>
+      <origin xyz="${fork_center_x} -0.25 -0.1885" rpy="0 0 0"/>
+      <geometry>
+        <box size="${fork_length} 0.10 0.04"/>
       </geometry>
       <material name="fork_gray"/>
     </visual>
     <collision name="fork_right_collision">
-      <origin xyz="-1.443 -0.25 -0.13" rpy="0 0 0"/>
-      <geometry>
-        <box size="1.20 0.10 0.04"/>
+      <origin xyz="${fork_center_x} -0.25 -0.1885" rpy="0 0 0"/>
+      <geometry>
+        <box size="${fork_length} 0.10 0.04"/>
       </geometry>
     </collision>
@@ -102,5 +113,5 @@
       <origin xyz="0 0 0" rpy="1.57079632679 0 0"/>
       <geometry>
-        <cylinder radius="${wheel_radius}" length="${wheel_width}"/>
+        <cylinder radius="${drive_wheel_radius}" length="${drive_wheel_width}"/>
       </geometry>
       <material name="wheel_black">
@@ -111,5 +122,5 @@
       <origin xyz="0 0 0" rpy="1.57079632679 0 0"/>
       <geometry>
-        <cylinder radius="${wheel_radius}" length="${wheel_width}"/>
+        <cylinder radius="${drive_wheel_radius}" length="${drive_wheel_width}"/>
       </geometry>
     </collision>
@@ -118,5 +129,5 @@
     <parent link="base_link"/>
     <child link="left_wheel_link"/>
-    <origin xyz="-0.34 ${wheel_separation / 2.0} -0.06" rpy="0 0 0"/>
+    <origin xyz="0 ${drive_track_width / 2.0} 0" rpy="0 0 0"/>
     <axis xyz="0 1 0"/>
   </joint>
@@ -130,5 +141,5 @@
       <origin xyz="0 0 0" rpy="1.57079632679 0 0"/>
       <geometry>
-        <cylinder radius="${wheel_radius}" length="${wheel_width}"/>
+        <cylinder radius="${drive_wheel_radius}" length="${drive_wheel_width}"/>
       </geometry>
       <material name="wheel_black"/>
@@ -137,5 +148,5 @@
       <origin xyz="0 0 0" rpy="1.57079632679 0 0"/>
       <geometry>
-        <cylinder radius="${wheel_radius}" length="${wheel_width}"/>
+        <cylinder radius="${drive_wheel_radius}" length="${drive_wheel_width}"/>
       </geometry>
     </collision>
@@ -144,16 +155,17 @@
     <parent link="base_link"/>
     <child link="right_wheel_link"/>
-    <origin xyz="-0.34 ${-wheel_separation / 2.0} -0.06" rpy="0 0 0"/>
+    <origin xyz="0 ${-drive_track_width / 2.0} 0" rpy="0 0 0"/>
     <axis xyz="0 1 0"/>
   </joint>
-  <link name="front_caster_link">
-    <inertial>
-      <origin xyz="0 0 0"/>
-      <mass value="0.4"/>
-      <inertia ixx="0.001" ixy="0.0" ixz="0.0" iyy="0.001" iyz="0.0" izz="0.001"/>
-    </inertial>
-    <visual>
-      <geometry>
-        <sphere radius="0.07"/>
+  <link name="left_support_wheel_link">
+    <inertial>
+      <origin xyz="0 0 0"/>
+      <mass value="1.0"/>
+      <inertia ixx="0.01" ixy="0.0" ixz="0.0" iyy="0.01" iyz="0.0" izz="0.01"/>
+    </inertial>
+    <visual>
+      <origin xyz="0 0 0" rpy="1.57079632679 0 0"/>
+      <geometry>
+        <cylinder radius="${support_wheel_radius}" length="${support_wheel_width}"/>
       </geometry>
       <material name="caster_dark">
@@ -162,13 +174,39 @@
     </visual>
     <collision>
-      <geometry>
-        <sphere radius="0.07"/>
-      </geometry>
-    </collision>
-  </link>
-  <joint name="front_caster_joint" type="fixed">
-    <parent link="base_link"/>
-    <child link="front_caster_link"/>
-    <origin xyz="0.42 0 -0.15" rpy="0 0 0"/>
+      <origin xyz="0 0 0" rpy="1.57079632679 0 0"/>
+      <geometry>
+        <cylinder radius="${support_wheel_radius}" length="${support_wheel_width}"/>
+      </geometry>
+    </collision>
+  </link>
+  <joint name="left_support_wheel_joint" type="fixed">
+    <parent link="base_link"/>
+    <child link="left_support_wheel_link"/>
+    <origin xyz="${wheel_base} ${support_track_width / 2.0} ${support_wheel_radius - drive_wheel_radius}" rpy="0 0 0"/>
+  </joint>
+  <link name="right_support_wheel_link">
+    <inertial>
+      <origin xyz="0 0 0"/>
+      <mass value="1.0"/>
+      <inertia ixx="0.01" ixy="0.0" ixz="0.0" iyy="0.01" iyz="0.0" izz="0.01"/>
+    </inertial>
+    <visual>
+      <origin xyz="0 0 0" rpy="1.57079632679 0 0"/>
+      <geometry>
+        <cylinder radius="${support_wheel_radius}" length="${support_wheel_width}"/>
+      </geometry>
+      <material name="caster_dark"/>
+    </visual>
+    <collision>
+      <origin xyz="0 0 0" rpy="1.57079632679 0 0"/>
+      <geometry>
+        <cylinder radius="${support_wheel_radius}" length="${support_wheel_width}"/>
+      </geometry>
+    </collision>
+  </link>
+  <joint name="right_support_wheel_joint" type="fixed">
+    <parent link="base_link"/>
+    <child link="right_support_wheel_link"/>
+    <origin xyz="${wheel_base} ${-support_track_width / 2.0} ${support_wheel_radius - drive_wheel_radius}" rpy="0 0 0"/>
   </joint>
   <link name="base_scan">
@@ -210,5 +248,10 @@
     <mu2>1.0</mu2>
   </gazebo>
-  <gazebo reference="front_caster_link">
+  <gazebo reference="left_support_wheel_link">
+    <material>Gazebo/Black</material>
+    <mu1>0.01</mu1>
+    <mu2>0.01</mu2>
+  </gazebo>
+  <gazebo reference="right_support_wheel_link">
     <material>Gazebo/Black</material>
     <mu1>0.01</mu1>
@@ -257,6 +300,6 @@
       <left_joint>left_wheel_joint</left_joint>
       <right_joint>right_wheel_joint</right_joint>
-      <wheel_separation>${wheel_separation}</wheel_separation>
-      <wheel_diameter>${2.0 * wheel_radius}</wheel_diameter>
+      <wheel_separation>${drive_track_width}</wheel_separation>
+      <wheel_diameter>${2.0 * drive_wheel_radius}</wheel_diameter>
       <max_wheel_torque>80</max_wheel_torque>
       <max_wheel_acceleration>1.0</max_wheel_acceleration>
